File: top_pcb/top_pcb.sch (KiCad schematic (older format))
At the start: 3 parts, among them J1 flat_cable_connector, J2 header, J3 free_holes

Commit message: Add hole to top_pcb
Parts:
- J3: footprint footprints:PinHeader_2x15_P2.54mm_Vertical_without_silks -> footprints:PinHeader_1x30_P1.27mm_Vertical_without_silks
Changed lines of the file:
@@
 EESchema Schematic File Version 4
 LIBS:top_pcb-cache
-EELAYER 26 0
+EELAYER 29 0
 EELAYER END
 $Descr A4 11693 8268
@@
 F 0 "J3" H 8150 3617 50  0000 C CNN
 F 1 "free_holes" H 8150 3526 50  0000 C CNN
-F 2 "footprints:PinHeader_2x15_P2.54mm_Vertical_without_silks" H 8100 2700 50  0001 C CNN
+F 2 "footprints:PinHeader_1x30_P1.27mm_Vertical_without_silks" H 8100 2700 50  0001 C CNN
 F 3 "~" H 8100 2700 50  0001 C CNN
 	1    8100 2700
